File: hardware/project/aurabip_preview.kicad_pcb (KiCad board)
At the start: 4 copper layers, 36 x 52 mm, 50 parts, among them J1 USB-C, J2 AKKU, J3 SPEAKER, J4 OLED, J5 u.FL 868, SW1 EIN/AUS, SW2 RESET, SW3 BOOT, U1 ESP32-S3-MINI-1, U10 E22-900M22S, U2 BMP581, U3 LSM6DSO32, U4 SHT40, U5 L96, U6 MAX98357A, U7 MCP73831, U8 AP2112K-3.3, U9 USBLC6

Commit message: fix(hardware): alle kritischen Pinouts gegen Datenblaetter verifiziert
Web-Recherche gegen Originalquellen (Ebyte Manual v1.3, Quectel HW
Design V1.4, ADI Rev 7, ST Rev 1) — drei von vier Annahmen waren falsch:
- E22-900M22S: 14x20/Pitch 1.27 statt 16x26/2.2, Pin-Map komplett neu
- L96: LCC-31 statt 12 Pads; RF-Bruecke R12 (RF_OUT->RF_IN, sonst kein
  GPS!), RXD-Pegelteiler R13/R14 (VIHmax 3.1V), C16, Antennen-Keepout
- MAX98357A: TQFN-Pinout neu (Pin 8 war VDD, nicht GND!), EP1.23-Footprint
- LSM6DSO32: Pinout bestaetigt, ST-Footprint statt Bosch (0.1mm-Versatz)

Dazu: Gehaeuse-Generator fuer Fusion 360 (hardware/fusion/, Varianten
audio/vision, Akku 504050, K-28-WP-Sitz, Antennen-Nische, Display-
Fenster), Board-STEP-Export, PCBWay-Fertigungspaket (export_fab.ps1 +
BOM-Generator), Akku auf 504050 1500mAh.

Co-Authored-By: Claude Fable 5 <noreply@anthropic.com>
Parts:
- J4: value OLED -> OLED SPI; footprint PinSocket_1x04_P2.54mm_Vertical -> JST_PH_B8B-PH-K_1x08_P2.00mm_Vertical
- moved SW2 23.2 mm to (47.0, 34.0)
- moved U2 21.1 mm to (47.5, 21.5)
- moved C4 19.1 mm to (45.5, 21.5), turned to 90 degrees
- moved U4 17.2 mm to (47.5, 25.0)
- moved C6 16.6 mm to (45.5, 25.0), turned to 90 degrees
- moved J2 16.0 mm to (47.0, 10.5)
- moved J3 16.0 mm to (47.0, 45.0)
- moved J4 6.80 mm to (38.0, 17.5), turned to 90 degrees
Connections:
- net LORA_MISO renamed SPI2_MISO
- J4 pad 3: I2C_SCL -> SPI2_MOSI
- J4 pad 4: I2C_SDA -> SPI2_SCK
- TP1 pad 1: TP_IO33 -> TP_IO38
- TP2 pad 1: TP_IO34 -> TP_IO40
- TP3 pad 1: TP_IO35 -> TP_IO41
- TP4 pad 1: TP_IO36 -> TP_IO42
- U1 pad 15: LORA_MOSI -> SPI2_MOSI
- U1 pad 16: LORA_SCK -> SPI2_SCK
- U1 pad 28: TP_IO33 -> OLED_CS
- U1 pad 29: TP_IO34 -> OLED_DC
- U1 pad 31: TP_IO35 -> OLED_RST
- U1 pad 32: TP_IO36 -> (no net)
- U1 pad 34: (no net) -> TP_IO38
- U1 pad 36: (no net) -> TP_IO40
- U1 pad 37: (no net) -> TP_IO41
- U1 pad 38: (no net) -> TP_IO42
- U10 pad 17: LORA_MOSI -> SPI2_MOSI
- U10 pad 18: LORA_SCK -> SPI2_SCK
Routing:
- net GND: track 25.7 -> 0.00 mm, vias 50 -> 0
- net +3V3: track 10.9 -> 0.00 mm, vias 20 -> 0
Other:
- board size 36 x 52 mm -> 52 x 52 mm
