File: hardware/project/aurabip_routed.kicad_pcb (KiCad board)
At the start: 4 copper layers, 52 x 52 mm, 53 parts, among them J1 USB-C, J2 AKKU, J3 SPEAKER, J4 OLED SPI, SW1 EIN/AUS, SW2 RESET, SW3 BOOT, U1 ESP32-S3-MINI-1, U10 E22-900M22S, U2 BMP581, U3 LSM6DSO32, U4 SHT40, U5 L96, U6 MAX98357A, U7 MCP73831, U8 AP2112K-3.3, U9 USBLC6

Commit message: wip(pcb): Via-in-Pad - 23/35 (GND-Stub-Handler ergaenzt), DRC 0/0
Routing:
- net GND: track 76.0 -> 77.9 mm, vias 82 -> 79
Changed lines of the file:
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@@
+	)
+	(segment
+		(start 24.985 23.522001)
+		(end 24.067414 23.713932)
+		(width 0.2)
+		(layer "F.Cu")
+		(net "GND")
 	)
 	(segment
@@
 	)
 	(segment
+		(start 45.5 21.02)
+		(end 45.8 20.7)
+		(width 0.2)
+		(layer "F.Cu")
+		(net "GND")
+	)
+	(segment
 		(start 24.075 4.3)
 		(end 26.123901 4.034843)
@@
 		(net "GND")
 	)
+	(segment
+		(start 45.5 24.52)
+		(end 45.5 24.02)
+		(width 0.2)
+		(layer "F.Cu")
+		(net "GND")
+	)
 	(via
 		(at 9.182001 18.514123)
@@
 	)
 	(via
-		(at 45.8 21.2)
-		(size 0.5)
-		(drill 0.3)
-		(layers "F.Cu" "B.Cu")
-		(net "GND")
-	)
-	(via
 		(at 26.123901 4.034843)
 		(size 0.5)
@@
 		(net "GND")
 	)
-	(via
-		(at 25.048618 23.243926)
-		(size 0.5)
-		(drill 0.3)
-		(layers "F.Cu" "B.Cu")
-		(locked yes)
-		(net "GND")
-	)
-	(via
-		(at 45.7 24.6)
-		(size 0.5)
-		(drill 0.3)
-		(layers "F.Cu" "B.Cu")
-		(net "GND")
-	)
